Commit message: try

File: src/adamu_description/urdf/adam_u.urdf (robot description, URDF)
Before this commit: robot adam_u, 51 links, 50 joints
Joints:
- joint left_wrist_to_tcp: origin xyz=0.0 0.0 -0.1 rpy=0 0 0 -> xyz=0.0 0.0 0.0 rpy=0 0 -3.14159; parent wristRollLeft -> left_hand_fts
- joint right_wrist_to_tcp: origin xyz=0.0 0.0 -0.1 rpy=0 0 0 -> xyz=0.0 0.0 0.0 rpy=0 0 0; parent wristRollRight -> right_hand_fts

File: src/adamu_moveit_config/config/adam_u.ros2_control.xacro (robot description, xacro)
@@ -168,4 +168,5 @@
             <joint name="shoulderPitch_Left">
                 <command_interface name="position"/>
+                <command_interface name="velocity"/>
                 <state_interface name="position">
                   <param name="initial_value">${initial_positions['shoulderPitch_Left']}</param>
@@ -175,4 +176,5 @@
             <joint name="shoulderRoll_Left">
                 <command_interface name="position"/>
+                <command_interface name="velocity"/>
                 <state_interface name="position">
                   <param name="initial_value">${initial_positions['shoulderRoll_Left']}</param>
@@ -182,4 +184,5 @@
             <joint name="shoulderYaw_Left">
                 <command_interface name="position"/>
+                <command_interface name="velocity"/>
                 <state_interface name="position">
                   <param name="initial_value">${initial_positions['shoulderYaw_Left']}</param>
@@ -189,4 +192,5 @@
             <joint name="elbow_Left">
                 <command_interface name="position"/>
+                <command_interface name="velocity"/>
                 <state_interface name="position">
                   <param name="initial_value">${initial_positions['elbow_Left']}</param>
@@ -196,4 +200,5 @@
             <joint name="wristYaw_Left">
                 <command_interface name="position"/>
+                <command_interface name="velocity"/>
                 <state_interface name="position">
                   <param name="initial_value">${initial_positions['wristYaw_Left']}</param>
@@ -203,4 +208,5 @@
             <joint name="wristPitch_Left">
                 <command_interface name="position"/>
+                <command_interface name="velocity"/>
                 <state_interface name="position">
                   <param name="initial_value">${initial_positions['wristPitch_Left']}</param>
@@ -210,4 +216,5 @@
             <joint name="wristRoll_Left">
                 <command_interface name="position"/>
+                <command_interface name="velocity"/>
                 <state_interface name="position">
                   <param name="initial_value">${initial_positions['wristRoll_Left']}</param>
@@ -217,4 +224,5 @@
             <joint name="shoulderPitch_Right">
                 <command_interface name="position"/>
+                <command_interface name="velocity"/>
                 <state_interface name="position">
                   <param name="initial_value">${initial_positions['shoulderPitch_Right']}</param>
@@ -224,4 +232,5 @@
             <joint name="shoulderRoll_Right">
                 <command_interface name="position"/>
+                <command_interface name="velocity"/>
                 <state_interface name="position">
                   <param name="initial_value">${initial_positions['shoulderRoll_Right']}</param>
@@ -231,4 +240,5 @@
             <joint name="shoulderYaw_Right">
                 <command_interface name="position"/>
+                <command_interface name="velocity"/>
                 <state_interface name="position">
                   <param name="initial_value">${initial_positions['shoulderYaw_Right']}</param>
@@ -238,4 +248,5 @@
             <joint name="elbow_Right">
                 <command_interface name="position"/>
+                <command_interface name="velocity"/>
                 <state_interface name="position">
                   <param name="initial_value">${initial_positions['elbow_Right']}</param>
@@ -245,4 +256,5 @@
             <joint name="wristYaw_Right">
                 <command_interface name="position"/>
+                <command_interface name="velocity"/>
                 <state_interface name="position">
                   <param name="initial_value">${initial_positions['wristYaw_Right']}</param>
@@ -252,4 +264,5 @@
             <joint name="wristPitch_Right">
                 <command_interface name="position"/>
+                <command_interface name="velocity"/>
                 <state_interface name="position">
                   <param name="initial_value">${initial_positions['wristPitch_Right']}</param>
@@ -259,4 +272,5 @@
             <joint name="wristRoll_Right">
                 <command_interface name="position"/>
+                <command_interface name="velocity"/>
                 <state_interface name="position">
                   <param name="initial_value">${initial_positions['wristRoll_Right']}</param>
@@ -266,4 +280,5 @@
             <joint name="L_index_MCP_joint">
                 <command_interface name="position"/>
+                <command_interface name="velocity"/>
                 <state_interface name="position">
                   <param name="initial_value">${initial_positions['L_index_MCP_joint']}</param>
@@ -273,4 +288,5 @@
             <joint name="L_index_DIP_joint">
                 <command_interface name="position"/>
+                <command_interface name="velocity"/>
                 <state_interface name="position">
                   <param name="initial_value">${initial_positions['L_index_DIP_joint']}</param>
@@ -280,4 +296,5 @@
             <joint name="L_middle_MCP_joint">
                 <command_interface name="position"/>
+                <command_interface name="velocity"/>
                 <state_interface name="position">
                   <param name="initial_value">${initial_positions['L_middle_MCP_joint']}</param>
@@ -287,4 +304,5 @@
             <joint name="L_middle_DIP_joint">
                 <command_interface name="position"/>
+                <command_interface name="velocity"/>
                 <state_interface name="position">
                   <param name="initial_value">${initial_positions['L_middle_DIP_joint']}</param>
@@ -294,4 +312,5 @@
             <joint name="L_pinky_MCP_joint">
                 <command_interface name="position"/>
+                <command_interface name="velocity"/>
                 <state_interface name="position">
                   <param name="initial_value">${initial_positions['L_pinky_MCP_joint']}</param>
@@ -301,4 +320,5 @@
             <joint name="L_pinky_DIP_joint">
                 <command_interface name="position"/>
+                <command_interface name="velocity"/>
                 <state_interface name="position">
                   <param name="initial_value">${initial_positions['L_pinky_DIP_joint']}</param>
@@ -308,4 +328,5 @@
             <joint name="L_ring_MCP_joint">
                 <command_interface name="position"/>
+                <command_interface name="velocity"/>
                 <state_interface name="position">
                   <param name="initial_value">${initial_positions['L_ring_MCP_joint']}</param>
@@ -315,4 +336,5 @@
             <joint name="L_ring_DIP_joint">
                 <command_interface name="position"/>
+                <command_interface name="velocity"/>
                 <state_interface name="position">
                   <param name="initial_value">${initial_positions['L_ring_DIP_joint']}</param>
@@ -322,4 +344,5 @@
             <joint name="L_thumb_MCP_joint1">
                 <command_interface name="position"/>
+                <command_interface name="velocity"/>
                 <state_interface name="position">
                   <param name="initial_value">${initial_positions['L_thumb_MCP_joint1']}</param>
@@ -329,4 +352,5 @@
             <joint name="L_thumb_MCP_joint2">
                 <command_interface name="position"/>
+                <command_interface name="velocity"/>
                 <state_interface name="position">
                   <param name="initial_value">${initial_positions['L_thumb_MCP_joint2']}</param>
@@ -336,4 +360,5 @@
             <joint name="L_thumb_PIP_joint">
                 <command_interface name="position"/>
+                <command_interface name="velocity"/>
                 <state_interface name="position">
                   <param name="initial_value">${initial_positions['L_thumb_PIP_joint']}</param>
@@ -343,4 +368,5 @@
             <joint name="L_thumb_DIP_joint">
                 <command_interface name="position"/>
+                <command_interface name="velocity"/>
                 <state_interface name="position">
                   <param name="initial_value">${initial_positions['L_thumb_DIP_joint']}</param>
@@ -350,4 +376,5 @@
             <joint name="R_index_MCP_joint">
                 <command_interface name="position"/>
+                <command_interface name="velocity"/>
                 <state_interface name="position">
                   <param name="initial_value">${initial_positions['R_index_MCP_joint']}</param>
@@ -357,4 +384,5 @@
             <joint name="R_index_DIP_joint">
                 <command_interface name="position"/>
+                <command_interface name="velocity"/>
                 <state_interface name="position">
                   <param name="initial_value">${initial_positions['R_index_DIP_joint']}</param>
@@ -364,4 +392,5 @@
             <joint name="R_middle_MCP_joint">
                 <command_interface name="position"/>
+                <command_interface name="velocity"/>
                 <state_interface name="position">
                   <param name="initial_value">${initial_positions['R_middle_MCP_joint']}</param>
@@ -371,4 +400,5 @@
             <joint name="R_middle_DIP_joint">
                 <command_interface name="position"/>
+                <command_interface name="velocity"/>
                 <state_interface name="position">
                   <param name="initial_value">${initial_positions['R_middle_DIP_joint']}</param>
@@ -378,4 +408,5 @@
             <joint name="R_pinky_MCP_joint">
                 <command_interface name="position"/>
+                <command_interface name="velocity"/>
                 <state_interface name="position">
                   <param name="initial_value">${initial_positions['R_pinky_MCP_joint']}</param>
@@ -385,4 +416,5 @@
             <joint name="R_pinky_DIP_joint">
                 <command_interface name="position"/>
+                <command_interface name="velocity"/>
                 <state_interface name="position">
                   <param name="initial_value">${initial_positions['R_pinky_DIP_joint']}</param>
@@ -392,4 +424,5 @@
             <joint name="R_ring_MCP_joint">
                 <command_interface name="position"/>
+                <command_interface name="velocity"/>
                 <state_interface name="position">
                   <param name="initial_value">${initial_positions['R_ring_MCP_joint']}</param>
@@ -399,4 +432,5 @@
             <joint name="R_ring_DIP_joint">
                 <command_interface name="position"/>
+                <command_interface name="velocity"/>
                 <state_interface name="position">
                   <param name="initial_value">${initial_positions['R_ring_DIP_joint']}</param>
@@ -406,4 +440,5 @@
             <joint name="R_thumb_MCP_joint1">
                 <command_interface name="position"/>
+                <command_interface name="velocity"/>
                 <state_interface name="position">
                   <param name="initial_value">${initial_positions['R_thumb_MCP_joint1']}</param>
@@ -413,4 +448,5 @@
             <joint name="R_thumb_MCP_joint2">
                 <command_interface name="position"/>
+                <command_interface name="velocity"/>
                 <state_interface name="position">
                   <param name="initial_value">${initial_positions['R_thumb_MCP_joint2']}</param>
@@ -420,4 +456,5 @@
             <joint name="R_thumb_PIP_joint">
                 <command_interface name="position"/>
+                <command_interface name="velocity"/>
                 <state_interface name="position">
                   <param name="initial_value">${initial_positions['R_thumb_PIP_joint']}</param>
@@ -427,4 +464,5 @@
             <joint name="R_thumb_DIP_joint">
                 <command_interface name="position"/>
+                <command_interface name="velocity"/>
                 <state_interface name="position">
                   <param name="initial_value">${initial_positions['R_thumb_DIP_joint']}</param>
@@ -434,4 +472,5 @@
             <joint name="waistRoll">
                 <command_interface name="position"/>
+                <command_interface name="velocity"/>
                 <state_interface name="position">
                   <param name="initial_value">${initial_positions['waistRoll']}</param>
@@ -441,4 +480,5 @@
             <joint name="waistPitch">
                 <command_interface name="position"/>
+                <command_interface name="velocity"/>
                 <state_interface name="position">
                   <param name="initial_value">${initial_positions['waistPitch']}</param>
@@ -448,4 +488,5 @@
             <joint name="waistYaw">
                 <command_interface name="position"/>
+                <command_interface name="velocity"/>
                 <state_interface name="position">
                   <param name="initial_value">${initial_positions['waistYaw']}</param>
@@ -455,4 +496,5 @@
             <joint name="neckYaw">
                 <command_interface name="position"/>
+                <command_interface name="velocity"/>
                 <state_interface name="position">
                   <param name="initial_value">${initial_positions['neckYaw']}</param>
@@ -462,4 +504,5 @@
             <joint name="neckPitch">
                 <command_interface name="position"/>
+                <command_interface name="velocity"/>
                 <state_interface name="position">
                   <param name="initial_value">${initial_positions['neckPitch']}</param>

Commit message: s

File: src/adamu_description/urdf/adam_u.urdf (robot description, URDF)
Before this commit: robot adam_u, 51 links, 50 joints
Joints:
- joint left_wrist_to_fts: origin xyz=0.0 0.0 -0.1 rpy=0 0 3.14159 -> xyz=0.0 0.0 -0.1 rpy=0 0 0
- joint left_wrist_to_tcp: origin xyz=0.0 0.0 0.0 rpy=0 0 -3.14159 -> xyz=0.0 0.0 0.0 rpy=0 0 0
